File: hsic-hub1.sch (KiCad schematic (older format))
At the start: 17 parts

Commit message: Major commit.
1. Fixed errors in libraries
2. Annoted schematics
3. Imported board shape and components into Pcbnew
Parts:
- removed C? (x3): 100n, Capacitor_SMD:C_0805_2012Metric_Pad1.15x1.40mm_HandSolder, symbol Drone:CAP
- removed C?: 1u, Capacitor_SMD:C_0805_2012Metric_Pad1.15x1.40mm_HandSolder, symbol Drone:CAP
- removed C?: 4u7, Capacitor_SMD:C_0805_2012Metric_Pad1.15x1.40mm_HandSolder, symbol Drone:CAP
- removed J? (x2): SM05B-SRSS-TB, Drone:SM05B-SRSS-TB, symbol Drone:SM05B-SRSS-TB
- removed R?: 10k, Resistor_SMD:R_0805_2012Metric_Pad1.15x1.40mm_HandSolder, symbol Drone:RES
- removed R?: DNP, Resistor_SMD:R_0805_2012Metric_Pad1.15x1.40mm_HandSolder, symbol Drone:RES
- removed U?: USB3503, symbol Drone:USB3503
- removed U?: TPS2054D, Package_SO:SOIC-16_3.9x9.9mm_P1.27mm, symbol Drone:TPS2054D
- added C35, C40, C41: 100n, Capacitor_SMD:C_0805_2012Metric, symbol Drone:CAP
- added C37: 4u7, Capacitor_SMD:C_0805_2012Metric, symbol Drone:CAP
- added C38: 1u, Capacitor_SMD:C_0805_2012Metric, symbol Drone:CAP
- added J14, J15: SM05B-SRSS-TB, Drone:SM05B-SRSS-TB, symbol Drone:SM05B-SRSS-TB
- added R39: DNP, Resistor_SMD:R_0805_2012Metric, symbol Drone:RES
- added R41: 10k, Resistor_SMD:R_0805_2012Metric, symbol Drone:RES
- added U10: TPS2054D, Package_SO:SOIC-16_3.9x9.9mm_P1.27mm, symbol Drone:TPS2054D
- added U9: USB3503, Drone:USB3503ML, symbol Drone:USB3503
- C34, C36, C39, C42: renamed from C?; footprint Capacitor_SMD:C_0805_2012Metric_Pad1.15x1.40mm_HandSolder -> Capacitor_SMD:C_0805_2012Metric
- R40: renamed from R?; footprint Resistor_SMD:R_0805_2012Metric_Pad1.15x1.40mm_HandSolder -> Resistor_SMD:R_0805_2012Metric
- gave numbers to parts that had none: 1
Changed lines of the file:
@@
 $Comp
 L Drone:USB3503 U?
-U 1 1 5E2F42C0
-P 5200 1050
-AR Path="/5E2B9068/5E2F42C0" Ref="U?"  Part="1"
-AR Path="/5E2EDC4D/5E2F42C0" Ref="U?"  Part="1"
-AR Path="/5E349830/5E2F42C0" Ref="U?"  Part="1"
-F 0 "U?" H 4600 1200 50  0000 L CNN
+U 1 1 5E888D16
+P 4600 1050
+AR Path="/5E2B9068/5E888D16" Ref="U?"  Part="1"
+AR Path="/5E2EDC4D/5E888D16" Ref="U?"  Part="1"
+AR Path="/5E349830/5E888D16" Ref="U9"  Part="1"
+F 0 "U9" H 4600 1200 50  0000 L CNN
 F 1 "USB3503" H 4600 1100 50  0000 L CNN
-F 2 "" H 5200 1050 50  0001 C CNN
-F 3 "http://www.microchip.com/mymicrochip/filehandler.aspx?ddocname=en566511" H 5200 1050 50  0001 C CNN
-	1    5200 1050
+F 2 "Drone:USB3503ML" H 4600 1050 50  0001 C CNN
+F 3 "http://www.microchip.com/mymicrochip/filehandler.aspx?ddocname=en566511" H 4600 1050 50  0001 C CNN
+	1    4600 1050
 	1    0    0    -1
 $EndComp
@@
 P 1150 5000
 AR Path="/5E2EDC4D/5E328065" Ref="C?"  Part="1"
-AR Path="/5E349830/5E328065" Ref="C?"  Part="1"
-F 0 "C?" H 1265 5046 50  0000 L CNN
+AR Path="/5E349830/5E328065" Ref="C34"  Part="1"
+F 0 "C34" H 1265 5046 50  0000 L CNN
 F 1 "100n" H 1265 4955 50  0000 L CNN
-F 2 "Capacitor_SMD:C_0805_2012Metric_Pad1.15x1.40mm_HandSolder" H 1188 4850 50  0001 C CNN
+F 2 "Capacitor_SMD:C_0805_2012Metric" H 1188 4850 50  0001 C CNN
 F 3 "~" H 1150 5000 50  0001 C CNN
 	1    1150 5000
@@
 $Comp
 L Drone:CAP C?
-U 1 1 5E332CF8
+U 1 1 5E888D1B
 P 9600 3500
-AR Path="/5E2EDC4D/5E332CF8" Ref="C?"  Part="1"
-AR Path="/5E349830/5E332CF8" Ref="C?"  Part="1"
-F 0 "C?" H 9715 3546 50  0000 L CNN
+AR Path="/5E2EDC4D/5E888D1B" Ref="C?"  Part="1"
+AR Path="/5E349830/5E888D1B" Ref="C41"  Part="1"
+F 0 "C41" H 9715 3546 50  0000 L CNN
 F 1 "100n" H 9715 3455 50  0000 L CNN
-F 2 "Capacitor_SMD:C_0805_2012Metric_Pad1.15x1.40mm_HandSolder" H 9638 3350 50  0001 C CNN
+F 2 "Capacitor_SMD:C_0805_2012Metric" H 9638 3350 50  0001 C CNN
 F 3 "~" H 9600 3500 50  0001 C CNN
 	1    9600 3500
@@
 P 1850 4850
 AR Path="/5E2EDC4D/5E308236" Ref="X?"  Part="1"
-AR Path="/5E349830/5E308236" Ref="X?"  Part="1"
-F 0 "X?" H 1650 5000 50  0000 L CNN
+AR Path="/5E349830/5E308236" Ref="X1"  Part="1"
+AR Path="/5E308236" Ref="X1"  Part="1"
+F 0 "X1" H 1650 5000 50  0000 L CNN
 F 1 "ASTXR-12" H 1650 4900 50  0000 L CNN
 F 2 "Drone:ASTXR-12" H 1650 4500 50  0001 L CNN
@@
 P 2400 5000
 AR Path="/5E2EDC4D/5E338829" Ref="C?"  Part="1"
-AR Path="/5E349830/5E338829" Ref="C?"  Part="1"
-F 0 "C?" H 2515 5046 50  0000 L CNN
+AR Path="/5E349830/5E338829" Ref="C36"  Part="1"
+F 0 "C36" H 2515 5046 50  0000 L CNN
 F 1 "1n" H 2515 4955 50  0000 L CNN
-F 2 "Capacitor_SMD:C_0805_2012Metric_Pad1.15x1.40mm_HandSolder" H 2438 4850 50  0001 C CNN
+F 2 "Capacitor_SMD:C_0805_2012Metric" H 2438 4850 50  0001 C CNN
 F 3 "~" H 2400 5000 50  0001 C CNN
 	1    2400 5000
@@
 P 9400 1350
 AR Path="/5E2EDC4D/5E3408C5" Ref="C?"  Part="1"
-AR Path="/5E349830/5E3408C5" Ref="C?"  Part="1"
-F 0 "C?" H 9515 1396 50  0000 L CNN
+AR Path="/5E349830/5E3408C5" Ref="C39"  Part="1"
+F 0 "C39" H 9515 1396 50  0000 L CNN
 F 1 "100n" H 9515 1305 50  0000 L CNN
-F 2 "Capacitor_SMD:C_0805_2012Metric_Pad1.15x1.40mm_HandSolder" H 9438 1200 50  0001 C CNN
+F 2 "Capacitor_SMD:C_0805_2012Metric" H 9438 1200 50  0001 C CNN
 F 3 "~" H 9400 1350 50  0001 C CNN
 	1    9400 1350
@@
 $Comp
 L Drone:CAP C?
-U 1 1 5E3AC9C8
+U 1 1 5E888D20
 P 9400 2350
-AR Path="/5E2EDC4D/5E3AC9C8" Ref="C?"  Part="1"
-AR Path="/5E349830/5E3AC9C8" Ref="C?"  Part="1"
-F 0 "C?" H 9515 2396 50  0000 L CNN
+AR Path="/5E2EDC4D/5E888D20" Ref="C?"  Part="1"
+AR Path="/5E349830/5E888D20" Ref="C40"  Part="1"
+F 0 "C40" H 9515 2396 50  0000 L CNN
 F 1 "100n" H 9515 2305 50  0000 L CNN
-F 2 "Capacitor_SMD:C_0805_2012Metric_Pad1.15x1.40mm_HandSolder" H 9438 2200 50  0001 C CNN
+F 2 "Capacitor_SMD:C_0805_2012Metric" H 9438 2200 50  0001 C CNN
 F 3 "~" H 9400 2350 50  0001 C CNN
 	1    9400 2350
@@
 $Comp
 L Drone:TPS2054D U?
-U 1 1 5E4E09E8
+U 1 1 5E888D23
 P 8550 3150
-AR Path="/5E2EDC4D/5E4E09E8" Ref="U?"  Part="1"
-AR Path="/5E349830/5E4E09E8" Ref="U?"  Part="1"
-F 0 "U?" H 8250 3300 50  0000 L BNN
+AR Path="/5E2EDC4D/5E888D23" Ref="U?"  Part="1"
+AR Path="/5E349830/5E888D23" Ref="U10"  Part="1"
+F 0 "U10" H 8250 3300 50  0000 L BNN
 F 1 "TPS2054D" H 8250 3200 50  0000 L BNN
 F 2 "Package_SO:SOIC-16_3.9x9.9mm_P1.27mm" H 8250 3400 50  0001 L BNN
@@
 $Comp
 L Drone:RES R?
-U 1 1 5E301315
+U 1 1 5E888D17
 P 7000 1600
-AR Path="/5E2EDC4D/5E301315" Ref="R?"  Part="1"
-AR Path="/5E349830/5E301315" Ref="R?"  Part="1"
-F 0 "R?" H 7070 1646 50  0000 L CNN
+AR Path="/5E2EDC4D/5E888D17" Ref="R?"  Part="1"
+AR Path="/5E349830/5E888D17" Ref="R41"  Part="1"
+F 0 "R41" H 7070 1646 50  0000 L CNN
 F 1 "10k" H 7070 1555 50  0000 L CNN
-F 2 "Resistor_SMD:R_0805_2012Metric_Pad1.15x1.40mm_HandSolder" V 6930 1600 50  0001 C CNN
+F 2 "Resistor_SMD:R_0805_2012Metric" V 6930 1600 50  0001 C CNN
 F 3 "~" H 7000 1600 50  0001 C CNN
 	1    7000 1600
@@
 $Comp
 L Drone:SM05B-SRSS-TB J?
-U 1 1 5E385FFC
+U 1 1 5E888D1E
 P 8500 1100
-AR Path="/5E2EDC4D/5E385FFC" Ref="J?"  Part="1"
-AR Path="/5E349830/5E385FFC" Ref="J?"  Part="1"
-F 0 "J?" H 8475 1000 50  0000 R CNN
+AR Path="/5E2EDC4D/5E888D1E" Ref="J?"  Part="1"
+AR Path="/5E349830/5E888D1E" Ref="J14"  Part="1"
+F 0 "J14" H 8475 1000 50  0000 R CNN
 F 1 "SM05B-SRSS-TB" H 8475 1075 50  0000 R CNN
 F 2 "Drone:SM05B-SRSS-TB" H 8350 1350 50  0001 L CNN
@@
 $Comp
 L Drone:SM05B-SRSS-TB J?
-U 1 1 5E3AC9C2
+U 1 1 5E888D1F
 P 8500 2100
-AR Path="/5E2EDC4D/5E3AC9C2" Ref="J?"  Part="1"
-AR Path="/5E349830/5E3AC9C2" Ref="J?"  Part="1"
-F 0 "J?" H 8475 2000 50  0000 R CNN
+AR Path="/5E2EDC4D/5E888D1F" Ref="J?"  Part="1"
+AR Path="/5E349830/5E888D1F" Ref="J15"  Part="1"
+F 0 "J15" H 8475 2000 50  0000 R CNN
 F 1 "SM05B-SRSS-TB" H 8475 2075 50  0000 R CNN
 F 2 "Drone:SM05B-SRSS-TB" H 8350 2350 50  0001 L CNN
@@
 P 10050 3500
 AR Path="/5E2EDC4D/5E5A610D" Ref="C?"  Part="1"
-AR Path="/5E349830/5E5A610D" Ref="C?"  Part="1"
-F 0 "C?" H 10165 3546 50  0000 L CNN
+AR Path="/5E349830/5E5A610D" Ref="C42"  Part="1"
+F 0 "C42" H 10165 3546 50  0000 L CNN
 F 1 "10u" H 10165 3455 50  0000 L CNN
-F 2 "Capacitor_SMD:C_0805_2012Metric_Pad1.15x1.40mm_HandSolder" H 10088 3350 50  0001 C CNN
+F 2 "Capacitor_SMD:C_0805_2012Metric" H 10088 3350 50  0001 C CNN
 F 3 "~" H 10050 3500 50  0001 C CNN
 	1    10050 3500
@@
 $Comp
 L Drone:CAP C?
-U 1 1 5E427B4C
+U 1 1 5E888D22
 P 2750 3550
-AR Path="/5E2EDC4D/5E427B4C" Ref="C?"  Part="1"
-AR Path="/5E349830/5E427B4C" Ref="C?"  Part="1"
-F 0 "C?" H 2865 3596 50  0000 L CNN
+AR Path="/5E2EDC4D/5E888D22" Ref="C?"  Part="1"
+AR Path="/5E349830/5E888D22" Ref="C37"  Part="1"
+F 0 "C37" H 2865 3596 50  0000 L CNN
 F 1 "4u7" H 2865 3505 50  0000 L CNN
-F 2 "Capacitor_SMD:C_0805_2012Metric_Pad1.15x1.40mm_HandSolder" H 2788 3400 50  0001 C CNN
+F 2 "Capacitor_SMD:C_0805_2012Metric" H 2788 3400 50  0001 C CNN
 F 3 "~" H 2750 3550 50  0001 C CNN
 	1    2750 3550
@@
 $Comp
 L Drone:CAP C?
-U 1 1 5E42226D
+U 1 1 5E888D21
 P 3150 3550
-AR Path="/5E2EDC4D/5E42226D" Ref="C?"  Part="1"
-AR Path="/5E349830/5E42226D" Ref="C?"  Part="1"
-F 0 "C?" H 3265 3596 50  0000 L CNN
+AR Path="/5E2EDC4D/5E888D21" Ref="C?"  Part="1"
+AR Path="/5E349830/5E888D21" Ref="C38"  Part="1"
+F 0 "C38" H 3265 3596 50  0000 L CNN
 F 1 "1u" H 3265 3505 50  0000 L CNN
-F 2 "Capacitor_SMD:C_0805_2012Metric_Pad1.15x1.40mm_HandSolder" H 3188 3400 50  0001 C CNN
+F 2 "Capacitor_SMD:C_0805_2012Metric" H 3188 3400 50  0001 C CNN
 F 3 "~" H 3150 3550 50  0001 C CNN
 	1    3150 3550
@@
 P 4200 3550
 AR Path="/5E2EDC4D/5E32A1DA" Ref="R?"  Part="1"
-AR Path="/5E349830/5E32A1DA" Ref="R?"  Part="1"
-F 0 "R?" H 4270 3596 50  0000 L CNN
+AR Path="/5E349830/5E32A1DA" Ref="R40"  Part="1"
+F 0 "R40" H 4270 3596 50  0000 L CNN
 F 1 "12k,1%" H 4270 3505 50  0000 L CNN
-F 2 "Resistor_SMD:R_0805_2012Metric_Pad1.15x1.40mm_HandSolder" V 4130 3550 50  0001 C CNN
+F 2 "Resistor_SMD:R_0805_2012Metric" V 4130 3550 50  0001 C CNN
 F 3 "~" H 4200 3550 50  0001 C CNN
 	1    4200 3550
@@
 $Comp
 L Drone:RES R?
-U 1 1 5E6510FD
+U 1 1 5E888D25
 P 2500 3050
-AR Path="/5E2EDC4D/5E6510FD" Ref="R?"  Part="1"
-AR Path="/5E349830/5E6510FD" Ref="R?"  Part="1"
-F 0 "R?" H 2570 3096 50  0000 L CNN
+AR Path="/5E2EDC4D/5E888D25" Ref="R?"  Part="1"
+AR Path="/5E349830/5E888D25" Ref="R39"  Part="1"
+F 0 "R39" H 2570 3096 50  0000 L CNN
 F 1 "DNP" H 2570 3005 50  0000 L CNN
-F 2 "Resistor_SMD:R_0805_2012Metric_Pad1.15x1.40mm_HandSolder" V 2430 3050 50  0001 C CNN
+F 2 "Resistor_SMD:R_0805_2012Metric" V 2430 3050 50  0001 C CNN
 F 3 "~" H 2500 3050 50  0001 C CNN
 	1    2500 3050
@@
 $Comp
 L Drone:CAP C?
-U 1 1 5E74B35F
+U 1 1 5E888D26
 P 2300 3550
-AR Path="/5E2EDC4D/5E74B35F" Ref="C?"  Part="1"
-AR Path="/5E349830/5E74B35F" Ref="C?"  Part="1"
-F 0 "C?" H 2415 3596 50  0000 L CNN
+AR Path="/5E2EDC4D/5E888D26" Ref="C?"  Part="1"
+AR Path="/5E349830/5E888D26" Ref="C35"  Part="1"
+F 0 "C35" H 2415 3596 50  0000 L CNN
 F 1 "100n" H 2415 3505 50  0000 L CNN
-F 2 "Capacitor_SMD:C_0805_2012Metric_Pad1.15x1.40mm_HandSolder" H 2338 3400 50  0001 C CNN
+F 2 "Capacitor_SMD:C_0805_2012Metric" H 2338 3400 50  0001 C CNN
 F 3 "~" H 2300 3550 50  0001 C CNN
 	1    2300 3550

Commit message: Work in progress on laying out the board.
Parts:
- C34, C35, C36, C37, C38, C39, C40, C41, C42: footprint Capacitor_SMD:C_0805_2012Metric -> Drone:C0805
- R39, R40, R41: footprint Resistor_SMD:R_0805_2012Metric -> Drone:R0805
Changed lines of the file:
@@
 F 0 "C34" H 1265 5046 50  0000 L CNN
 F 1 "100n" H 1265 4955 50  0000 L CNN
-F 2 "Capacitor_SMD:C_0805_2012Metric" H 1188 4850 50  0001 C CNN
+F 2 "Drone:C0805" H 1188 4850 50  0001 C CNN
 F 3 "~" H 1150 5000 50  0001 C CNN
 	1    1150 5000
@@
 F 0 "C41" H 9715 3546 50  0000 L CNN
 F 1 "100n" H 9715 3455 50  0000 L CNN
-F 2 "Capacitor_SMD:C_0805_2012Metric" H 9638 3350 50  0001 C CNN
+F 2 "Drone:C0805" H 9638 3350 50  0001 C CNN
 F 3 "~" H 9600 3500 50  0001 C CNN
 	1    9600 3500
@@
 F 0 "C36" H 2515 5046 50  0000 L CNN
 F 1 "1n" H 2515 4955 50  0000 L CNN
-F 2 "Capacitor_SMD:C_0805_2012Metric" H 2438 4850 50  0001 C CNN
+F 2 "Drone:C0805" H 2438 4850 50  0001 C CNN
 F 3 "~" H 2400 5000 50  0001 C CNN
 	1    2400 5000
@@
 F 0 "C39" H 9515 1396 50  0000 L CNN
 F 1 "100n" H 9515 1305 50  0000 L CNN
-F 2 "Capacitor_SMD:C_0805_2012Metric" H 9438 1200 50  0001 C CNN
+F 2 "Drone:C0805" H 9438 1200 50  0001 C CNN
 F 3 "~" H 9400 1350 50  0001 C CNN
 	1    9400 1350
@@
 F 0 "C40" H 9515 2396 50  0000 L CNN
 F 1 "100n" H 9515 2305 50  0000 L CNN
-F 2 "Capacitor_SMD:C_0805_2012Metric" H 9438 2200 50  0001 C CNN
+F 2 "Drone:C0805" H 9438 2200 50  0001 C CNN
 F 3 "~" H 9400 2350 50  0001 C CNN
 	1    9400 2350
@@
 F 0 "R41" H 7070 1646 50  0000 L CNN
 F 1 "10k" H 7070 1555 50  0000 L CNN
-F 2 "Resistor_SMD:R_0805_2012Metric" V 6930 1600 50  0001 C CNN
+F 2 "Drone:R0805" V 6930 1600 50  0001 C CNN
 F 3 "~" H 7000 1600 50  0001 C CNN
 	1    7000 1600
@@
 F 0 "C42" H 10165 3546 50  0000 L CNN
 F 1 "10u" H 10165 3455 50  0000 L CNN
-F 2 "Capacitor_SMD:C_0805_2012Metric" H 10088 3350 50  0001 C CNN
+F 2 "Drone:C0805" H 10088 3350 50  0001 C CNN
 F 3 "~" H 10050 3500 50  0001 C CNN
 	1    10050 3500
@@
 F 0 "C37" H 2865 3596 50  0000 L CNN
 F 1 "4u7" H 2865 3505 50  0000 L CNN
-F 2 "Capacitor_SMD:C_0805_2012Metric" H 2788 3400 50  0001 C CNN
+F 2 "Drone:C0805" H 2788 3400 50  0001 C CNN
 F 3 "~" H 2750 3550 50  0001 C CNN
 	1    2750 3550
@@
 F 0 "C38" H 3265 3596 50  0000 L CNN
 F 1 "1u" H 3265 3505 50  0000 L CNN
-F 2 "Capacitor_SMD:C_0805_2012Metric" H 3188 3400 50  0001 C CNN
+F 2 "Drone:C0805" H 3188 3400 50  0001 C CNN
 F 3 "~" H 3150 3550 50  0001 C CNN
 	1    3150 3550
@@
 F 0 "R40" H 4270 3596 50  0000 L CNN
 F 1 "12k,1%" H 4270 3505 50  0000 L CNN
-F 2 "Resistor_SMD:R_0805_2012Metric" V 4130 3550 50  0001 C CNN
+F 2 "Drone:R0805" V 4130 3550 50  0001 C CNN
 F 3 "~" H 4200 3550 50  0001 C CNN
 	1    4200 3550
@@
 F 0 "R39" H 2570 3096 50  0000 L CNN
 F 1 "DNP" H 2570 3005 50  0000 L CNN
-F 2 "Resistor_SMD:R_0805_2012Metric" V 2430 3050 50  0001 C CNN
+F 2 "Drone:R0805" V 2430 3050 50  0001 C CNN
 F 3 "~" H 2500 3050 50  0001 C CNN
 	1    2500 3050
@@
 F 0 "C35" H 2415 3596 50  0000 L CNN
 F 1 "100n" H 2415 3505 50  0000 L CNN
-F 2 "Capacitor_SMD:C_0805_2012Metric" H 2338 3400 50  0001 C CNN
+F 2 "Drone:C0805" H 2338 3400 50  0001 C CNN
 F 3 "~" H 2300 3550 50  0001 C CNN
 	1    2300 3550

Commit message: Many the minor updates.
Parts:
- added R35: 10k, Drone:R0805, symbol Drone:RES
Connections:
- net PRTPWR: now also R41.2
- net VDD33_BYP: now also R35.1
- net ~OSC: now also R35.2; no longer R41.2
Changed lines of the file:
@@
 Text Label 10450 3250 2    50   ~ 0
 5V
-Wire Wire Line
-	6000 1900 6700 1900
 $Comp
 L Drone:CAP C?
@@
 Wire Wire Line
 	7700 3650 8050 3650
-Wire Wire Line
-	7000 1000 7000 1450
-Wire Wire Line
-	6000 2050 7000 2050
-$Comp
-L Drone:RES R?
-U 1 1 5E888D17
-P 7000 1600
-AR Path="/5E2EDC4D/5E888D17" Ref="R?"  Part="1"
-AR Path="/5E349830/5E888D17" Ref="R41"  Part="1"
-F 0 "R41" H 7070 1646 50  0000 L CNN
-F 1 "10k" H 7070 1555 50  0000 L CNN
-F 2 "Drone:R0805" V 6930 1600 50  0001 C CNN
-F 3 "~" H 7000 1600 50  0001 C CNN
-	1    7000 1600
-	1    0    0    -1
-$EndComp
-Wire Wire Line
-	7000 2050 7000 1750
 $Comp
 L Drone:SM05B-SRSS-TB J?
@@
 Wire Wire Line
 	2750 2850 2750 3400
-Text Label 7000 1000 3    50   ~ 0
-VDD33_BYP
 Wire Wire Line
 	2300 1150 2300 3400
@@
 Text Label 2300 4100 1    50   ~ 0
 GND
+Wire Wire Line
+	7000 1000 7000 1450
+$Comp
+L Drone:RES R?
+U 1 1 5E59E0D7
+P 7000 1600
+AR Path="/5E2EDC4D/5E59E0D7" Ref="R?"  Part="1"
+AR Path="/5E349830/5E59E0D7" Ref="R41"  Part="1"
+F 0 "R41" H 7070 1646 50  0000 L CNN
+F 1 "10k" H 7070 1555 50  0000 L CNN
+F 2 "Drone:R0805" V 6930 1600 50  0001 C CNN
+F 3 "~" H 7000 1600 50  0001 C CNN
+	1    7000 1600
+	1    0    0    -1
+$EndComp
+Text Label 7000 1000 3    50   ~ 0
+VDD33_BYP
+Wire Wire Line
+	7300 1000 7300 1450
+$Comp
+L Drone:RES R?
+U 1 1 5E59E0DF
+P 7300 1600
+AR Path="/5E2EDC4D/5E59E0DF" Ref="R?"  Part="1"
+AR Path="/5E349830/5E59E0DF" Ref="R35"  Part="1"
+F 0 "R35" H 7370 1646 50  0000 L CNN
+F 1 "10k" H 7370 1555 50  0000 L CNN
+F 2 "Drone:R0805" V 7230 1600 50  0001 C CNN
+F 3 "~" H 7300 1600 50  0001 C CNN
+	1    7300 1600
+	1    0    0    -1
+$EndComp
+Text Label 7300 1000 3    50   ~ 0
+VDD33_BYP
+Wire Wire Line
+	7300 2050 7300 1750
+Wire Wire Line
+	6000 2050 7300 2050
+Wire Wire Line
+	7000 1900 7000 1750
+Wire Wire Line
+	6000 1900 7000 1900
 $EndSCHEMATC

Commit message: Update layout
Parts:
- U10: footprint Package_SO:SOIC-16_3.9x9.9mm_P1.27mm -> Drone:TPS2054D
- renumbered J14 to J12, J15 to J16
Changed lines of the file:
@@
 F 0 "U10" H 8250 3300 50  0000 L BNN
 F 1 "TPS2054D" H 8250 3200 50  0000 L BNN
-F 2 "Package_SO:SOIC-16_3.9x9.9mm_P1.27mm" H 8250 3400 50  0001 L BNN
+F 2 "Drone:TPS2054D" H 8250 3400 50  0001 L BNN
 F 3 "" H 8500 3150 50  0001 C CNN
 	1    8550 3150
@@
 P 8500 1100
 AR Path="/5E2EDC4D/5E888D1E" Ref="J?"  Part="1"
-AR Path="/5E349830/5E888D1E" Ref="J14"  Part="1"
-F 0 "J14" H 8475 1000 50  0000 R CNN
+AR Path="/5E349830/5E888D1E" Ref="J12"  Part="1"
+F 0 "J12" H 8475 1000 50  0000 R CNN
 F 1 "SM05B-SRSS-TB" H 8475 1075 50  0000 R CNN
 F 2 "Drone:SM05B-SRSS-TB" H 8350 1350 50  0001 L CNN
@@
 P 8500 2100
 AR Path="/5E2EDC4D/5E888D1F" Ref="J?"  Part="1"
-AR Path="/5E349830/5E888D1F" Ref="J15"  Part="1"
-F 0 "J15" H 8475 2000 50  0000 R CNN
+AR Path="/5E349830/5E888D1F" Ref="J16"  Part="1"
+F 0 "J16" H 8475 2000 50  0000 R CNN
 F 1 "SM05B-SRSS-TB" H 8475 2075 50  0000 R CNN
 F 2 "Drone:SM05B-SRSS-TB" H 8350 2350 50  0001 L CNN

Commit message: Use standard names for differential pair nets.
Connections:
- net USB1_DM renamed USB3_DN
- net USB1_DP renamed USB3_DP
- net USB2_DM renamed USB4_DN
- net USB2_DP renamed USB4_DP
Changed lines of the file:
@@
 Wire Wire Line
 	9050 3550 9400 3550
-Text Label 7700 1250 0    50   ~ 0
-USB1_DM
-Text Label 7700 1350 0    50   ~ 0
-USB1_DP
 Text Label 9400 3450 2    50   ~ 0
 USB1_5V
@@
 	1    0    0    -1
 $EndComp
-Text Label 7700 2250 0    50   ~ 0
-USB2_DM
-Text Label 7700 2350 0    50   ~ 0
-USB2_DP
 Text Label 7700 2150 0    50   ~ 0
 USB2_5V
@@
 	8100 2700 8100 2550
 Text Label 6700 1500 2    50   ~ 0
-USB1_DM
+USB3_DN
 Text Label 6700 1400 2    50   ~ 0
-USB1_DP
+USB3_DP
 Wire Wire Line
 	6000 1400 6700 1400
@@
 	6000 1500 6700 1500
 Text Label 6700 1750 2    50   ~ 0
-USB2_DM
+USB4_DN
 Text Label 6700 1650 2    50   ~ 0
-USB2_DP
+USB4_DP
 Wire Wire Line
 	6000 1650 6700 1650
@@
 Wire Wire Line
 	6000 1900 7000 1900
+Text Label 7700 1350 0    50   ~ 0
+USB3_DP
+Text Label 7700 1250 0    50   ~ 0
+USB3_DN
+Text Label 7700 2350 0    50   ~ 0
+USB4_DP
+Text Label 7700 2250 0    50   ~ 0
+USB4_DN
 $EndSCHEMATC

Commit message: Work in progress commit (component placement)
Connections:
- net USB1_5V renamed USB3_5V
- net USB2_5V renamed USB4_5V
Changed lines of the file:
@@
 	9050 3550 9400 3550
 Text Label 9400 3450 2    50   ~ 0
-USB1_5V
+USB3_5V
 Text Label 9400 3550 2    50   ~ 0
-USB2_5V
+USB4_5V
 Text Label 7700 1150 0    50   ~ 0
-USB1_5V
+USB3_5V
 Text Label 7700 1550 0    50   ~ 0
 GND
@@
 $EndComp
 Text Label 7700 2150 0    50   ~ 0
-USB2_5V
+USB4_5V
 Text Label 7700 2550 0    50   ~ 0
 GND

Commit message: Major commit 1. Moved a couple components and rerouted accordingly 2. Added fabrication information to all components 3. Several clean ups to footprints 4. Removed some unused components
Parts:
- U10: value TPS2054D -> TPS2054BDR; footprint Drone:TPS2054D -> Drone:TPS2054BDR; symbol Drone:TPS2054D -> Drone:TPS2054BDR
Changed lines of the file:
@@
 ~OSC
 $Comp
-L Drone:TPS2054D U?
+L Drone:TPS2054BDR U?
 U 1 1 5E888D23
 P 8550 3150
 AR Path="/5E2EDC4D/5E888D23" Ref="U?"  Part="1"
 AR Path="/5E349830/5E888D23" Ref="U10"  Part="1"
+AR Path="/5E888D23" Ref="U10"  Part="1"
 F 0 "U10" H 8250 3300 50  0000 L BNN
-F 1 "TPS2054D" H 8250 3200 50  0000 L BNN
-F 2 "Drone:TPS2054D" H 8250 3400 50  0001 L BNN
+F 1 "TPS2054BDR" H 8250 3200 50  0000 L BNN
+F 2 "Drone:TPS2054BDR" H 8250 3400 50  0001 L BNN
 F 3 "" H 8500 3150 50  0001 C CNN
 	1    8550 3150
