File: power.sch (KiCad schematic (older format))
At the start: 17 parts

Commit message: Updates to schematic library and power circuitry.
Parts:
- removed Q?: BSS138DW, symbol Drone:BSS138DW
- removed R? (x2): 10k, Resistor_SMD:R_0805_2012Metric_Pad1.15x1.40mm_HandSolder, symbol Drone:RES
- removed U?: TLV75528PDBV, Package_TO_SOT_SMD:SOT-23-5, symbol Regulator_Linear:TLV75528PDBV
- removed U?: TLV75518PDBV, Package_TO_SOT_SMD:SOT-23-5, symbol Regulator_Linear:TLV75518PDBV
- added R?: 1k, Resistor_SMD:R_0805_2012Metric_Pad1.15x1.40mm_HandSolder, symbol Drone:RES
- added S?: ES02MSABE, symbol Drone:ES02MSABE
- added U?: TLV75518PDBV, Package_TO_SOT_SMD:SOT-23-5, symbol Drone:TLV75518PDBV
- added U?: TLV75528PDBV, Package_TO_SOT_SMD:SOT-23-5, symbol Drone:TLV75528PDBV
- C? (x4): value 10u -> 1u
- U?: footprint (none) -> Drone:D36V28F3
Connections:
- net labels added: MTR_EN_18, ~PMU_SLP_18
- net labels removed: GPIO_CTR?_18, GPIO_CTR?_33
- wire segments 85 -> 74
- no-connect marks 0 -> 4
Other:
- note added: "Power Board Connector"
- note added: "TODO: EN after 5V is good and not SLP"
- note added: "TODO: Pull down CTRL unless switched"
- note removed: "1. PG low battery indicator? (open drain and external pull up resistor is required)\n2. Enabled by default so EN shouldnt be wired?\n3. any capacitors missing?"
- note removed: "1. capacitors are within min and max in datasheet (but why choose what value?)\n2. EN is higher than V_HI (more than 1V) (check!)\n3. when i copy them to copter lib (many variations are copied as well!)"
- note removed: "Motor_Driver_Connector"
- moved on the sheet: C?, J?, Q?A, R?, SSR?, U?

Commit message: Minor tweaks to schematics.
Parts:
- added Q?: BSS138DW, symbol Drone:BSS138DW
Connections:
- net at U?.2 (EN): now also Q?.6 (D2)
Changed lines of the file:
@@
 	9300 3350 8650 3350
 Text Label 8650 3450 0    50   ~ 0
-~PMU_SLP_18
+SYS_EN_18
 Text Label 8650 3350 0    50   ~ 0
 MTR_EN_18
@@
 Text Notes 4700 1600 0    50   ~ 0
 TODO: EN after 5V is good and not SLP
+$Comp
+L Drone:BSS138DW Q?
+U 1 1 5E456F98
+P 4300 2750
+AR Path="/5E2EDC4D/5E456F98" Ref="Q?"  Part="1"
+AR Path="/5E456F98" Ref="Q?"  Part="1"
+AR Path="/5E3E92F4/5E456F98" Ref="Q?"  Part="1"
+F 0 "Q?" V 4550 2650 50  0000 L CNN
+F 1 "BSS138DW" V 4450 2650 50  0000 L CNN
+F 2 "" H 4400 2675 50  0001 L CIN
+F 3 "https://www.diodes.com/assets/Datasheets/ds30203.pdf" H 4200 2750 50  0001 L CNN
+	1    4300 2750
+	1    0    0    -1
+$EndComp
+Wire Wire Line
+	4600 2100 4300 2100
+Wire Wire Line
+	4300 2100 4300 2550
+Text Label 3700 3150 0    50   ~ 0
+SYS_EN_18
 $EndSCHEMATC

Commit message: Finalized power schematic.
Parts:
- removed Q?: BSS138DW, symbol Drone:BSS138DW
- removed R? (x2): 10k, Resistor_SMD:R_0805_2012Metric_Pad1.15x1.40mm_HandSolder, symbol Drone:RES
- added Q? (x3): BSS138DW, symbol Drone:BSS138DW
- added R?: 100k, Resistor_SMD:R_0805_2012Metric_Pad1.15x1.40mm_HandSolder, symbol Drone:RES
- added R?: 10k, Resistor_SMD:R_0805_2012Metric_Pad1.15x1.40mm_HandSolder, symbol Drone:RES
- added R?: 5.6k, Resistor_SMD:R_0805_2012Metric_Pad1.15x1.40mm_HandSolder, symbol Drone:RES
Connections:
- net GPIO_MTR?_3V3 is gone; now on net 3V3: U?.3 (CTRL+)
- net 11V1: now also R?.1
- net 5V: now also R?.1
- net GND: now also Q?.1 (S2), Q?.4 (S2), Q?.4 (S2), R?.2; no longer U?.4 (CTRL-)
- net MTR_EN_18: now also Q?.5 (G2)
- net at Q?.2 (G2): now also Q?.6 (D2), R?.2
- new net: Q?.3 (D2), U?.4 (CTRL-)
- new net: Q?.1 (S2), Q?.3 (D2)
- new net: Q?.2 (G2), R?.1, R?.2
- new net SYS_EN_18: Q?.5 (G2)
Other:
- note removed: "TODO: EN after 5V is good and not SLP"
- note removed: "TODO: Pull down CTRL unless switched"
- moved on the sheet: C?, J?, Q?A, R?, S?, SSR?, U?

Commit message: Major commit.
1. Fixed errors in libraries
2. Annoted schematics
3. Imported board shape and components into Pcbnew
Parts:
- C52, C53, C54, C55: renamed from C?; footprint Capacitor_SMD:C_0805_2012Metric_Pad1.15x1.40mm_HandSolder -> Capacitor_SMD:C_0805_2012Metric
- Q6, Q7: renamed from Q?; footprint (none) -> Package_TO_SOT_SMD:SOT-363_SC-70-6
- R45, R46, R47, R48: renamed from R?; footprint Resistor_SMD:R_0805_2012Metric_Pad1.15x1.40mm_HandSolder -> Resistor_SMD:R_0805_2012Metric
- S1: renamed from S?; footprint (none) -> Drone:ES02MSABE
- U13: renamed from U?; footprint Drone:D36V50F5 -> Drone:D36V50F5_S
- U14: renamed from U?; footprint Drone:D36V28F3 -> Drone:D36V28F3_S
- gave numbers to parts that had none: 5
Connections:
- no-connect marks 4 -> 3
Changed lines of the file:
@@
 P 10400 2150
 AR Path="/5E349830/5E4477E2" Ref="C?"  Part="1"
-AR Path="/5E3E92F4/5E4477E2" Ref="C?"  Part="1"
-F 0 "C?" H 10515 2196 50  0000 L CNN
+AR Path="/5E3E92F4/5E4477E2" Ref="C55"  Part="1"
+F 0 "C55" H 10515 2196 50  0000 L CNN
 F 1 "1u" H 10515 2105 50  0000 L CNN
-F 2 "Capacitor_SMD:C_0805_2012Metric_Pad1.15x1.40mm_HandSolder" H 10438 2000 50  0001 C CNN
+F 2 "Capacitor_SMD:C_0805_2012Metric" H 10438 2000 50  0001 C CNN
 F 3 "~" H 10400 2150 50  0001 C CNN
 	1    10400 2150
@@
 P 9000 2150
 AR Path="/5E349830/5E4477D8" Ref="C?"  Part="1"
-AR Path="/5E3E92F4/5E4477D8" Ref="C?"  Part="1"
-F 0 "C?" H 9115 2196 50  0000 L CNN
+AR Path="/5E3E92F4/5E4477D8" Ref="C54"  Part="1"
+F 0 "C54" H 9115 2196 50  0000 L CNN
 F 1 "1u" H 9115 2105 50  0000 L CNN
-F 2 "Capacitor_SMD:C_0805_2012Metric_Pad1.15x1.40mm_HandSolder" H 9038 2000 50  0001 C CNN
+F 2 "Capacitor_SMD:C_0805_2012Metric" H 9038 2000 50  0001 C CNN
 F 3 "~" H 9000 2150 50  0001 C CNN
 	1    9000 2150
@@
 P 8400 2150
 AR Path="/5E349830/5E41DB5A" Ref="C?"  Part="1"
-AR Path="/5E3E92F4/5E41DB5A" Ref="C?"  Part="1"
-F 0 "C?" H 8515 2196 50  0000 L CNN
+AR Path="/5E3E92F4/5E41DB5A" Ref="C53"  Part="1"
+F 0 "C53" H 8515 2196 50  0000 L CNN
 F 1 "1u" H 8515 2105 50  0000 L CNN
-F 2 "Capacitor_SMD:C_0805_2012Metric_Pad1.15x1.40mm_HandSolder" H 8438 2000 50  0001 C CNN
+F 2 "Capacitor_SMD:C_0805_2012Metric" H 8438 2000 50  0001 C CNN
 F 3 "~" H 8400 2150 50  0001 C CNN
 	1    8400 2150
@@
 P 7000 2150
 AR Path="/5E349830/5E40BD7D" Ref="C?"  Part="1"
-AR Path="/5E3E92F4/5E40BD7D" Ref="C?"  Part="1"
-F 0 "C?" H 7115 2196 50  0000 L CNN
+AR Path="/5E3E92F4/5E40BD7D" Ref="C52"  Part="1"
+F 0 "C52" H 7115 2196 50  0000 L CNN
 F 1 "1u" H 7115 2105 50  0000 L CNN
-F 2 "Capacitor_SMD:C_0805_2012Metric_Pad1.15x1.40mm_HandSolder" H 7038 2000 50  0001 C CNN
+F 2 "Capacitor_SMD:C_0805_2012Metric" H 7038 2000 50  0001 C CNN
 F 3 "~" H 7000 2150 50  0001 C CNN
 	1    7000 2150
@@
 3V3
 $Comp
-L Drone:XT60PW-F_Vertical J?
+L Drone:XT60PW-F_Vertical J18
 U 1 1 5E3DE251
 P 9800 3750
-F 0 "J?" H 9600 3425 50  0000 L CNN
+F 0 "J18" H 9600 3425 50  0000 L CNN
 F 1 "XT60PW-F_Vertical" H 9600 3500 50  0000 L CNN
 F 2 "Drone:XT60-F_1x02_P7.20mm_Vertical" H 9700 4000 50  0001 L BNN
@@
 $EndComp
 $Comp
-L Drone:XT90PW-M J?
+L Drone:XT90PW-M J19
 U 1 1 5E3D24EA
 P 9800 4800
-F 0 "J?" H 9693 4433 50  0000 C CNN
+F 0 "J19" H 9693 4433 50  0000 C CNN
 F 1 "XT90PW-M" H 9693 4524 50  0000 C CNN
 F 2 "Drone:XT90PW-M" H 9700 5050 50  0001 L BNN
@@
 P 5550 1750
 AR Path="/5E3B18FA" Ref="U?"  Part="1"
-AR Path="/5E3E92F4/5E3B18FA" Ref="U?"  Part="1"
-F 0 "U?" H 5550 1850 50  0000 L BNN
+AR Path="/5E3E92F4/5E3B18FA" Ref="U14"  Part="1"
+F 0 "U14" H 5550 1850 50  0000 L BNN
 F 1 "D36V28F3" H 5550 1775 50  0000 L BNN
-F 2 "Drone:D36V28F3" H 5500 1700 50  0001 C CNN
+F 2 "Drone:D36V28F3_S" H 5500 1700 50  0001 C CNN
 F 3 "https://www.pololu.com/product/3781" H 5500 1700 50  0001 C CNN
 	1    5550 1750
@@
 P 2250 1750
 AR Path="/5E3ABE9B" Ref="U?"  Part="1"
-AR Path="/5E3E92F4/5E3ABE9B" Ref="U?"  Part="1"
-F 0 "U?" H 2250 1850 50  0000 L BNN
+AR Path="/5E3E92F4/5E3ABE9B" Ref="U13"  Part="1"
+F 0 "U13" H 2250 1850 50  0000 L BNN
 F 1 "D36V50F5" H 2250 1775 50  0000 L BNN
-F 2 "Drone:D36V50F5" H 2200 1700 50  0001 C CNN
+F 2 "Drone:D36V50F5_S" H 2200 1700 50  0001 C CNN
 F 3 "https://www.pololu.com/product/4091" H 2200 1700 50  0001 C CNN
 	1    2250 1750
@@
 P 8600 3500
 AR Path="/5E3F8AD0" Ref="SSR?"  Part="1"
-AR Path="/5E3E92F4/5E3F8AD0" Ref="U?"  Part="1"
-F 0 "U?" H 8400 3625 50  0000 C CNN
+AR Path="/5E3E92F4/5E3F8AD0" Ref="U16"  Part="1"
+F 0 "U16" H 8400 3625 50  0000 C CNN
 F 1 "CMX60D20" H 8550 3550 50  0000 C CNN
 F 2 "Drone:CMX60D20" H 8500 3500 50  0001 L BNN
@@
 MTR_EN_18
 $Comp
-L Drone:TLV75518PDBV U?
+L Drone:TLV75518PDBV U17
 U 1 1 5E58F736
 P 9500 1750
-F 0 "U?" H 9500 1850 50  0000 L BNN
+F 0 "U17" H 9500 1850 50  0000 L BNN
 F 1 "TLV75518PDBV" H 9500 1775 50  0000 L BNN
 F 2 "Package_TO_SOT_SMD:SOT-23-5" H 9500 2050 50  0001 C CIN
@@
 $EndComp
 $Comp
-L Drone:TLV75528PDBV U?
+L Drone:TLV75528PDBV U15
 U 1 1 5E59019E
 P 7500 1750
-F 0 "U?" H 7500 1850 50  0000 L BNN
+F 0 "U15" H 7500 1850 50  0000 L BNN
 F 1 "TLV75528PDBV" H 7500 1775 50  0000 L BNN
 F 2 "Package_TO_SOT_SMD:SOT-23-5" H 7500 2050 50  0001 C CIN
@@
 Wire Wire Line
 	2950 1850 3150 1850
-NoConn ~ 5450 2150
 NoConn ~ 2150 2450
 Text Label 4350 1850 0    50   ~ 0
@@
 GND
 $Comp
-L Drone:ES02MSABE S?
+L Drone:ES02MSABE S1
 U 1 1 5E69A4C6
 P 1350 2250
-F 0 "S?" H 1350 2350 50  0000 L BNN
+F 0 "S1" H 1350 2350 50  0000 L BNN
 F 1 "ES02MSABE" H 1350 2275 50  0000 L BNN
-F 2 "" H 1575 2150 50  0001 C CNN
+F 2 "Drone:ES02MSABE" H 1575 2150 50  0001 C CNN
 F 3 "https://dznh3ojzb2azq.cloudfront.net/products/Slide/ES/documents/datasheet.pdf" H 1500 2150 50  0001 C CNN
 	1    1350 2250
@@
 AR Path="/5E2EDC4D/5E6ACD3A" Ref="R?"  Part="1"
 AR Path="/5E6ACD3A" Ref="R?"  Part="1"
-AR Path="/5E3E92F4/5E6ACD3A" Ref="R?"  Part="1"
-F 0 "R?" H 1170 2646 50  0000 L CNN
+AR Path="/5E3E92F4/5E6ACD3A" Ref="R45"  Part="1"
+F 0 "R45" H 1170 2646 50  0000 L CNN
 F 1 "1k" H 1170 2555 50  0000 L CNN
-F 2 "Resistor_SMD:R_0805_2012Metric_Pad1.15x1.40mm_HandSolder" V 1030 2600 50  0001 C CNN
+F 2 "Resistor_SMD:R_0805_2012Metric" V 1030 2600 50  0001 C CNN
 F 3 "~" H 1100 2600 50  0001 C CNN
 	1    1100 2600
@@
 AR Path="/5E2EDC4D/5E456F98" Ref="Q?"  Part="1"
 AR Path="/5E456F98" Ref="Q?"  Part="1"
-AR Path="/5E3E92F4/5E456F98" Ref="Q?"  Part="1"
-F 0 "Q?" V 5400 3100 50  0000 L CNN
+AR Path="/5E3E92F4/5E456F98" Ref="Q7"  Part="1"
+F 0 "Q7" V 5400 3100 50  0000 L CNN
 F 1 "BSS138DW" V 5300 3100 50  0000 L CNN
-F 2 "" H 5250 3125 50  0001 L CIN
+F 2 "Package_TO_SOT_SMD:SOT-363_SC-70-6" H 5250 3125 50  0001 L CIN
 F 3 "https://www.diodes.com/assets/Datasheets/ds30203.pdf" H 5050 3200 50  0001 L CNN
 	1    5150 3200
@@
 AR Path="/5E2EDC4D/5E4B6163" Ref="R?"  Part="1"
 AR Path="/5E4B6163" Ref="R?"  Part="1"
-AR Path="/5E3E92F4/5E4B6163" Ref="R?"  Part="1"
-F 0 "R?" H 4770 2646 50  0000 L CNN
+AR Path="/5E3E92F4/5E4B6163" Ref="R48"  Part="1"
+F 0 "R48" H 4770 2646 50  0000 L CNN
 F 1 "100k" H 4770 2555 50  0000 L CNN
-F 2 "Resistor_SMD:R_0805_2012Metric_Pad1.15x1.40mm_HandSolder" V 4630 2600 50  0001 C CNN
+F 2 "Resistor_SMD:R_0805_2012Metric" V 4630 2600 50  0001 C CNN
 F 3 "~" H 4700 2600 50  0001 C CNN
 	1    4700 2600
@@
 AR Path="/5E2EDC4D/5E4C65D5" Ref="Q?"  Part="2"
 AR Path="/5E4C65D5" Ref="Q?"  Part="2"
-AR Path="/5E3E92F4/5E4C65D5" Ref="Q?"  Part="2"
-F 0 "Q?" V 4650 4050 50  0000 L CNN
+AR Path="/5E3E92F4/5E4C65D5" Ref="Q6"  Part="2"
+F 0 "Q6" V 4650 4050 50  0000 L CNN
 F 1 "BSS138DW" V 4550 4050 50  0000 L CNN
-F 2 "" H 4500 4075 50  0001 L CIN
+F 2 "Package_TO_SOT_SMD:SOT-363_SC-70-6" H 4500 4075 50  0001 L CIN
 F 3 "https://www.diodes.com/assets/Datasheets/ds30203.pdf" H 4300 4150 50  0001 L CNN
 	2    4400 4150
@@
 AR Path="/5E2EDC4D/5E4D7614" Ref="Q?"  Part="1"
 AR Path="/5E4D7614" Ref="Q?"  Part="1"
-AR Path="/5E3E92F4/5E4D7614" Ref="Q?"  Part="1"
-F 0 "Q?" V 4650 3550 50  0000 L CNN
+AR Path="/5E3E92F4/5E4D7614" Ref="Q6"  Part="1"
+F 0 "Q6" V 4650 3550 50  0000 L CNN
 F 1 "BSS138DW" V 4550 3550 50  0000 L CNN
-F 2 "" H 4500 3575 50  0001 L CIN
+F 2 "Package_TO_SOT_SMD:SOT-363_SC-70-6" H 4500 3575 50  0001 L CIN
 F 3 "https://www.diodes.com/assets/Datasheets/ds30203.pdf" H 4300 3650 50  0001 L CNN
 	1    4400 3650
@@
 AR Path="/5E2EDC4D/5E57AB75" Ref="Q?"  Part="2"
 AR Path="/5E57AB75" Ref="Q?"  Part="2"
-AR Path="/5E3E92F4/5E57AB75" Ref="Q?"  Part="2"
-F 0 "Q?" V 8150 4000 50  0000 L CNN
+AR Path="/5E3E92F4/5E57AB75" Ref="Q7"  Part="2"
+F 0 "Q7" V 8150 4000 50  0000 L CNN
 F 1 "BSS138DW" V 8050 4000 50  0000 L CNN
-F 2 "" H 8000 4025 50  0001 L CIN
+F 2 "Package_TO_SOT_SMD:SOT-363_SC-70-6" H 8000 4025 50  0001 L CIN
 F 3 "https://www.diodes.com/assets/Datasheets/ds30203.pdf" H 7800 4100 50  0001 L CNN
 	2    7900 4100
@@
 AR Path="/5E2EDC4D/5E5A9908" Ref="R?"  Part="1"
 AR Path="/5E5A9908" Ref="R?"  Part="1"
-AR Path="/5E3E92F4/5E5A9908" Ref="R?"  Part="1"
-F 0 "R?" H 3320 3446 50  0000 L CNN
+AR Path="/5E3E92F4/5E5A9908" Ref="R46"  Part="1"
+F 0 "R46" H 3320 3446 50  0000 L CNN
 F 1 "10k" H 3320 3355 50  0000 L CNN
-F 2 "Resistor_SMD:R_0805_2012Metric_Pad1.15x1.40mm_HandSolder" V 3180 3400 50  0001 C CNN
+F 2 "Resistor_SMD:R_0805_2012Metric" V 3180 3400 50  0001 C CNN
 F 3 "~" H 3250 3400 50  0001 C CNN
 	1    3250 3400
@@
 AR Path="/5E2EDC4D/5E5A9BE0" Ref="R?"  Part="1"
 AR Path="/5E5A9BE0" Ref="R?"  Part="1"
-AR Path="/5E3E92F4/5E5A9BE0" Ref="R?"  Part="1"
-F 0 "R?" H 3320 3946 50  0000 L CNN
+AR Path="/5E3E92F4/5E5A9BE0" Ref="R47"  Part="1"
+F 0 "R47" H 3320 3946 50  0000 L CNN
 F 1 "5.6k" H 3320 3855 50  0000 L CNN
-F 2 "Resistor_SMD:R_0805_2012Metric_Pad1.15x1.40mm_HandSolder" V 3180 3900 50  0001 C CNN
+F 2 "Resistor_SMD:R_0805_2012Metric" V 3180 3900 50  0001 C CNN
 F 3 "~" H 3250 3900 50  0001 C CNN
 	1    3250 3900

Commit message: Work in progress on laying out the board.
Parts:
- C52, C53, C54, C55: footprint Capacitor_SMD:C_0805_2012Metric -> Drone:C0805
- R45, R46, R47, R48: footprint Resistor_SMD:R_0805_2012Metric -> Drone:R0805
Changed lines of the file:
@@
 F 0 "C55" H 10515 2196 50  0000 L CNN
 F 1 "1u" H 10515 2105 50  0000 L CNN
-F 2 "Capacitor_SMD:C_0805_2012Metric" H 10438 2000 50  0001 C CNN
+F 2 "Drone:C0805" H 10438 2000 50  0001 C CNN
 F 3 "~" H 10400 2150 50  0001 C CNN
 	1    10400 2150
@@
 F 0 "C54" H 9115 2196 50  0000 L CNN
 F 1 "1u" H 9115 2105 50  0000 L CNN
-F 2 "Capacitor_SMD:C_0805_2012Metric" H 9038 2000 50  0001 C CNN
+F 2 "Drone:C0805" H 9038 2000 50  0001 C CNN
 F 3 "~" H 9000 2150 50  0001 C CNN
 	1    9000 2150
@@
 F 0 "C53" H 8515 2196 50  0000 L CNN
 F 1 "1u" H 8515 2105 50  0000 L CNN
-F 2 "Capacitor_SMD:C_0805_2012Metric" H 8438 2000 50  0001 C CNN
+F 2 "Drone:C0805" H 8438 2000 50  0001 C CNN
 F 3 "~" H 8400 2150 50  0001 C CNN
 	1    8400 2150
@@
 F 0 "C52" H 7115 2196 50  0000 L CNN
 F 1 "1u" H 7115 2105 50  0000 L CNN
-F 2 "Capacitor_SMD:C_0805_2012Metric" H 7038 2000 50  0001 C CNN
+F 2 "Drone:C0805" H 7038 2000 50  0001 C CNN
 F 3 "~" H 7000 2150 50  0001 C CNN
 	1    7000 2150
@@
 F 0 "R45" H 1170 2646 50  0000 L CNN
 F 1 "1k" H 1170 2555 50  0000 L CNN
-F 2 "Resistor_SMD:R_0805_2012Metric" V 1030 2600 50  0001 C CNN
+F 2 "Drone:R0805" V 1030 2600 50  0001 C CNN
 F 3 "~" H 1100 2600 50  0001 C CNN
 	1    1100 2600
@@
 F 0 "R48" H 4770 2646 50  0000 L CNN
 F 1 "100k" H 4770 2555 50  0000 L CNN
-F 2 "Resistor_SMD:R_0805_2012Metric" V 4630 2600 50  0001 C CNN
+F 2 "Drone:R0805" V 4630 2600 50  0001 C CNN
 F 3 "~" H 4700 2600 50  0001 C CNN
 	1    4700 2600
@@
 F 0 "R46" H 3320 3446 50  0000 L CNN
 F 1 "10k" H 3320 3355 50  0000 L CNN
-F 2 "Resistor_SMD:R_0805_2012Metric" V 3180 3400 50  0001 C CNN
+F 2 "Drone:R0805" V 3180 3400 50  0001 C CNN
 F 3 "~" H 3250 3400 50  0001 C CNN
 	1    3250 3400
@@
 F 0 "R47" H 3320 3946 50  0000 L CNN
 F 1 "5.6k" H 3320 3855 50  0000 L CNN
-F 2 "Resistor_SMD:R_0805_2012Metric" V 3180 3900 50  0001 C CNN
+F 2 "Drone:R0805" V 3180 3900 50  0001 C CNN
 F 3 "~" H 3250 3900 50  0001 C CNN
 	1    3250 3900

Commit message: Update layout
Changed lines of the file:
@@
 AR Path="/5E3F8AD0" Ref="SSR?"  Part="1"
 AR Path="/5E3E92F4/5E3F8AD0" Ref="U16"  Part="1"
-F 0 "U16" H 8400 3625 50  0000 C CNN
+F 0 "U16" H 8350 3600 50  0000 L BNN
 F 1 "CMX60D20" H 8550 3550 50  0000 C CNN
 F 2 "Drone:CMX60D20" H 8500 3500 50  0001 L BNN
